File: hardware/v2/gpsdo.brd (EAGLE design)
At the start: 76.2 x 69.8 mm, 80 parts, among them IC1 74HCT125N, IC2 74HCT125N, IC3 78L05, IC5 78L09, Q2 2N2222, U1 LMC6482DIL, U2 MAR-4, U3 MAR-4

Commit message: Rename components
Parts:
- removed PROGRAM: (no value), SparkFun:1X03
- removed SV1: (no value), SparkFun-Connectors:1X04
- added J1: (no value), SparkFun-Connectors:1X01
- added J2: (no value), SparkFun-Connectors:1X06
- added LED5: R/G, led:LED3MM
- added R19: 5.1K, resistor:0207/2V
- C1, C3: value 390pF -> .1uF; device zener:CAP-PTH-SMALL -> SparkFun:CAP-PTH-SMALL
- C10: value 4.7uF -> 390pF; device SparkFun-Capacitors:EIA3216 -> zener:CAP-PTH-SMALL
- C11: value .33uF -> 680pF; device SparkFun-Capacitors:CAP-PTH-SMALL -> zener:CAP-PTH-SMALL
- C12, C4: value .1uF -> 390pF; device SparkFun:CAP-PTH-SMALL -> zener:CAP-PTH-SMALL
- C13: device SparkFun-Capacitors:CAP-PTH-SMALL -> SparkFun-Capacitors:CAP-PTH-5MM
- C14: value .1uF -> 1uF; device SparkFun:CAP-PTH-SMALL -> SparkFun-Passives:CAP-PTH-SMALL
- C15: value 4.7uF -> 1uF; device SparkFun-Capacitors:EIA3216 -> SparkFun-Passives:CAP-PTH-SMALL
- C16: value .1uF -> .001uF; device SparkFun-Capacitors:CAP-PTH-5MM -> SparkFun-Capacitors:CAP-PTH-SMALL
- C17: value .1uF -> 4.7uF; device SparkFun-Capacitors:CAP-PTH-SMALL -> SparkFun-Capacitors:EIA3216
- C18: value .001uF -> .33uF
- C2: value 680pF -> .1uF; device zener:CAP-PTH-SMALL -> SparkFun:CAP-PTH-SMALL
- C21, C23: device SparkFun:CAP-PTH-SMALL -> SparkFun-Capacitors:CAP-PTH-SMALL
- C22: value 10uF -> .33uF; device SparkFun-Passives:CPOL-RADIAL-10UF-25V -> SparkFun-Capacitors:CAP-PTH-SMALL
- C24: value 390pF -> .1uF; device zener:CAP-PTH-SMALL -> SparkFun-Capacitors:CAP-PTH-SMALL
- C25: value 680pF -> 10uF; device zener:CAP-PTH-SMALL -> SparkFun-Passives:CPOL-RADIAL-10UF-25V
- C26: value 390pF -> 4.7uF; device zener:CAP-PTH-SMALL -> SparkFun-Capacitors:EIA3216
- C27: value .01uF -> .33uF
- C28: value .33uF -> .01uF
- C29: value .33uF -> .1uF
- C5: value .1uF -> 680pF; device SparkFun:CAP-PTH-SMALL -> zener:CAP-PTH-SMALL
- C6: value 1uF -> 390pF; device SparkFun-Passives:CAP-PTH-SMALL -> zener:CAP-PTH-SMALL
- C7: value 1uF -> .1uF; device SparkFun-Passives:CAP-PTH-SMALL -> SparkFun:CAP-PTH-SMALL
- C8, C9: device SparkFun-Capacitors:CAP-PTH-SMALL -> SparkFun:CAP-PTH-SMALL
- IC1: device 74xx-us:DIL14 -> 74xx-eu:DIL14
- IC2: device 74xx-eu:DIL14 -> 74xx-us:DIL14
- JP1, JP2: value (none) -> M02PTH; device SparkFun-Connectors:1X06 -> SparkFun-Connectors:1X02
- JP11: device SparkFun-Connectors:1X04 -> SparkFun:1X02
- JP4: device SparkFun:1X02 -> SparkFun-Connectors:1X04@1
- JP5, JP6: device SparkFun:1X03 -> SparkFun-Connectors:1X06@1
- JP7: value M02PTH -> (none); device SparkFun-Connectors:1X02 -> SparkFun:1X05
- JP8: device SparkFun:1X05 -> SparkFun:1X03
- JP9: value M02PTH -> (none); device SparkFun-Connectors:1X02 -> SparkFun:1X03
- LED1: value YELLOW -> GREEN
- LED2: value GREEN -> YELLOW
- R10: value 10K -> 0; device resistor:RTRIM3296W -> resistor:0207/2V
- R11: value 47K -> 1k
- R12: value 1k -> 330
- R13: value 6.8k -> 100K
- R14: value 10k -> 100K
- R17: value 5.1K -> 47K
- R4: value 100K -> 10K; device resistor:0207/2V -> resistor:RTRIM3296W
- R5: value 100K -> 75
- R6: value 0 -> 330
- R7: value 75 -> 330
- R8: value 330 -> 6.8k
- R9: value 330 -> 10k
- U1: value LMC6482DIL -> MAR-4; device overby:DIL08 -> LTC3200:VV105
- U3: value MAR-4 -> LMC6482DIL; device LTC3200:VV105 -> overby:DIL08
- moved R12 68.7 mm to (68.6, 10.2), turned to 270 degrees
- moved R9 66.5 mm to (11.4, 40.6)
- moved C25 66.4 mm to (8.26, 12.1)
- moved R8 64.8 mm to (11.4, 44.5), turned to 0 degrees
- moved C8 64.5 mm to (36.8, 66.0), turned to 180 degrees
- moved C10 63.7 mm to (39.4, 66.0), turned to 270 degrees
- moved JP7 61.4 mm to (27.9, 3.81), turned to 0 degrees
- moved C26 61.2 mm to (8.89, 25.4), turned to 0 degrees
- moved C11 59.9 mm to (47.0, 66.0), turned to 270 degrees
- moved R7 57.9 mm to (68.6, 15.2)
- moved C9 57.5 mm to (57.1, 63.5), turned to 90 degrees
- moved C21 52.6 mm to (12.1, 10.8)
- moved JP2 51.4 mm to (72.4, 47.0), turned to 90 degrees
- moved JP11 50.8 mm to (3.81, 24.8), turned to 90 degrees
- moved JP10 50.6 mm to (39.4, 20.3), turned to 0 degrees
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- renumbered Q2 to Q1, SJ2 to SJ1, U$1 to IC$1, U$3 to L3, U$4 to L1, U$5 to L2, U$6 to L4
Connections:
- removed net N$8: JP6.3, Q1.3, R18.1
- new net N$28: LED5.A, R16.1
- new net N$29: J1.1, R16.2
- net +3V3: now also C23.1, C24.1, IC2.14, R17.2, R2.2, R4.1; no longer C17.1, C9.1, IC1.14, R10.3, R11.2, R3.2
- net +5V: now also C17.A, C19.1, IC1.14, J2.3, JP5.3, JP7.2; no longer C10.A, C8.1, IC2.14, JP11.2, JP2.3, JP8.2
- net +9V: now also C26.A, C28.1, C29.1, R5.2; no longer C13.1, C15.A, C27.1, R7.2
- net 1PPS: now also IC2.6, JP8.3; no longer IC1.6, JP5.3
- net 1PPSIN: now also IC2.5, JP7.5; no longer IC1.5, JP8.5
- net CLOCK: now also IC2.11, IC2.9; no longer IC1.11, IC1.9
- net GND: now also C10.2, C12.2, C14.2, C15.2, C17.C, C21.2, C23.2, C26.C, C4.2, C5.2, J2.1, JP11.2, JP4.3, JP5.1, LED5.K, R3.1, R4.3, R9.2, U1.2; no longer C1.2, C10.C, C15.C, C17.2, C2.2, C26.2, C3.2, C7.2, C8.2, C9.2, JP11.1, JP4.2, JP8.1, PROGRAM.1, R10.1, R14.2, R2.1, SV1.3, U3.2
- net GOODLED: now also IC1.12; no longer IC2.12
- net GPSLOCK: now also IC2.3; no longer IC1.3
- net GPSRXI: now also JP5.4, JP7.4; no longer JP2.4, JP8.4
- net GPSTXO: now also J2.4, JP5.5, JP7.3; no longer JP11.3, JP2.5, JP8.3
- net LOCK-IN: now also IC2.2, J2.5; no longer IC1.2, JP11.4
- net LOCKLED: now also IC1.5; no longer IC2.5
- net N$1: now also LED2.A, R7.1; no longer LED1.A, R8.1
- net N$10: now also C2.2, U1.3; no longer C21.2, U2.3
- net N$11: now also C3.1, IC2.12, R2.1, R3.2, R4.2; no longer C5.1, IC1.12, R10.2, R2.2, R3.1
- net N$12: now also LED1.A, R6.1; no longer LED2.A, R9.1
- net N$13: now also R11.2, R8.1, U3.7; no longer R12.2, R13.1, U1.7
- net N$14: now also C1.2, C7.2, JP1.2; no longer C12.2, C4.2, JP7.2
- net N$15: now also R10.2, U3.2; no longer R6.2, U1.2
- net N$16: now also C11.1; no longer C25.1
- net N$17: now also JP11.1; no longer JP4.1
- net N$18: now also C12.1, C9.2; no longer C14.2, C26.1
- net N$19: now also JP10.2; no longer JP9.2
- net N$2: now also C5.1; no longer C2.1
- net N$20: now also IC1.8, R12.2; no longer IC2.8, R15.2
- net N$21: now also IC1.11, R15.2; no longer IC2.11, R16.2
- net N$22: now also C8.2, R5.1, U2.3; no longer C23.2, R7.1, U3.3
- net N$23: now also C16.1, JP9.2, R17.1; no longer C18.1, PROGRAM.2, R11.1
- net N$24: now also C10.1, C8.1; no longer C23.1, C24.1
- net N$25: now also C7.1, U2.1; no longer C12.1, U3.1
- net N$26: now also C9.1, JP3.2; no longer C14.1, JP10.2
- net N$27: now also JP9.3; no longer PROGRAM.3
- net N$3: now also C3.2, C6.1; no longer C3.1, C5.2
- net N$30: now also IC2.8, JP2.2; no longer IC1.8, JP3.2
- net N$31: now also C13.1, U3.8; no longer C16.1, U1.8
- net N$33: now also C2.1, C4.1; no longer C1.1, C21.1
- net N$35: now also IC1.3, R6.2; no longer IC2.3, R9.2
- net N$36: now also IC1.6, R7.2; no longer IC2.6, R8.2
- net N$37: now also R8.2, R9.1, U3.6; no longer R13.2, R14.1, U1.6
- net N$39: now also R12.1; no longer R15.1
- net N$4: now also C1.1, U1.1; no longer C4.1, U2.1
- net N$40: now also R15.1; no longer R16.1
- net N$41: now also R19.2; no longer R17.2
- net N$5: now also C14.1, R13.1, U3.5; no longer C7.1, R5.1, U1.5
- net N$6: now also R10.1, R13.2, U3.1; no longer R5.2, R6.1, U1.1
- net N$7: now also C15.1, R14.1, U3.3; no longer C6.1, R4.1, U1.3
- net N$9: now also JP8.2; no longer JP5.2
- net OSC-HEATER: now also JP4.4, R19.1; no longer R17.1, SV1.4
- net OSCH: now also Q1.3, R18.1; no longer JP6.2
- net PWRIN: now also C18.1, C21.1, C25.1, C27.1; no longer C11.1, C19.1, C28.1, C29.1
- net PWRLED: now also IC1.9; no longer IC2.9
- net RXIN: now also JP6.4, JP8.1; no longer JP1.4, JP5.1
- net STATUSLED: now also IC1.2; no longer IC2.2
- net TXOUT: now also JP6.5; no longer JP1.5
- net VCOADJUST: now also JP4.1, R11.1; no longer R12.1, SV1.1
- net VCOPWM: now also R14.2; no longer R4.2
- net VCOPWR: now also JP4.2; no longer SV1.2
Routing:
- net GND: track 368.7 -> 343.0 mm
- net OSCH: track 24.2 -> 34.9 mm
- net N$35: track 26.5 -> 16.3 mm, vias 1 -> 0
- net N$20: track 13.8 -> 3.81 mm
- net N$8: track 8.67 -> 0.00 mm
- net +5V: track 115.7 -> 123.8 mm
- net +3V3: track 117.9 -> 122.4 mm
- net LOCK-IN: track 41.5 -> 45.8 mm
- net RXIN: track 5.61 -> 9.72 mm
- net N$36: track 17.6 -> 14.3 mm
- net N$9: track 9.72 -> 6.66 mm
- net N$29: track 0.00 -> 3.07 mm
- net 1PPSIN: track 54.6 -> 51.6 mm, vias 3 -> 0
- net N$28: track 0.00 -> 2.54 mm
- net TXOUT: track 15.8 -> 13.2 mm
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Other:
- board text added: "v2.1"
- board text added: "© Copyright Glen Overby 2014-2017"
- board text removed: "Copyright Glen Overby 2014-2016"
- board text removed: "OSCready"
- board text removed: "v2.0"
